Commit message: Initial commit or updated package

File: urdf/dyno_atman.urdf.xacro (robot description, xacro)
@@ -1,4 +1,5 @@
 <?xml version="1.0"?>
 <robot name="my_mesh_robot" xmlns:xacro="http://www.ros.org/wiki/xacro">
+  <!-- Base footprint -->
   <link name="base_footprint"/>
   <joint name="base_joint" type="fixed">
@@ -7,11 +8,18 @@
     <origin xyz="0 0 0.1075" rpy="0 0 0"/>
   </joint>
+  <!-- BASE LINK -->
   <link name="base_link">
     <visual>
-      <geometry><mesh filename="package://gazebo/meshes/base_link.STL"/></geometry>
-      <material name="grey"><color rgba="0.5 0.5 0.5 1"/></material>
-    </visual>
-    <collision>
-      <geometry><mesh filename="package://gazebo/meshes/base_link.STL"/></geometry>
+      <geometry>
+        <mesh filename="package://gazebo/meshes/base_link.STL"/>
+      </geometry>
+      <material name="grey">
+        <color rgba="0.5 0.5 0.5 1"/>
+      </material>
+    </visual>
+    <collision>
+      <geometry>
+        <mesh filename="package://gazebo/meshes/base_link.STL"/>
+      </geometry>
     </collision>
     <inertial>
@@ -20,12 +28,19 @@
     </inertial>
   </link>
+  <!-- LEFT WHEEL -->
   <link name="left_wheel">
     <visual>
       <origin xyz="0 0 0" rpy="1.5708 0 0"/>
-      <geometry><mesh filename="package://gazebo/meshes/l_wheel.STL"/></geometry>
-      <material name="black"><color rgba="0 0 0 1"/></material>
-    </visual>
-    <collision>
-      <geometry><cylinder radius="0.1075" length="0.05"/></geometry>
+      <geometry>
+        <mesh filename="package://gazebo/meshes/l_wheel.STL"/>
+      </geometry>
+      <material name="black">
+        <color rgba="0 0 0 1"/>
+      </material>
+    </visual>
+    <collision>
+      <geometry>
+        <cylinder radius="0.1075" length="0.05"/>
+      </geometry>
     </collision>
     <inertial>
@@ -41,12 +56,19 @@
     <dynamics damping="1.0" friction="0.2"/>
   </joint>
+  <!-- RIGHT WHEEL -->
   <link name="right_wheel">
     <visual>
       <origin xyz="0 0 0" rpy="1.5708 0 0"/>
-      <geometry><mesh filename="package://gazebo/meshes/r_wheel.STL"/></geometry>
-      <material name="black"/>
-    </visual>
-    <collision>
-      <geometry><cylinder radius="0.1075" length="0.05"/></geometry>
+      <geometry>
+        <mesh filename="package://gazebo/meshes/r_wheel.STL"/>
+      </geometry>
+      <material name="black">
+        <color rgba="0 0 0 1"/>
+      </material>
+    </visual>
+    <collision>
+      <geometry>
+        <cylinder radius="0.1075" length="0.05"/>
+      </geometry>
     </collision>
     <inertial>
@@ -62,5 +84,5 @@
     <dynamics damping="1.0" friction="0.2"/>
   </joint>
-  <!-- Friction / contact for wheels (important: on the link collision, not the joint) -->
+  <!-- WHEEL FRICTION -->
   <gazebo reference="left_wheel">
     <collision>
@@ -68,5 +90,4 @@
         <friction>
           <ode>
-          <!-- increase friction to reduce slip -->
             <mu>1.2</mu>
             <mu2>1.2</mu2>
@@ -75,5 +96,4 @@
         <contact>
           <ode>
-          <!-- stiffer contact to avoid interpenetration + reduce jitter/slip -->
             <kp>50000</kp>
             <kd>1.0</kd>
@@ -101,11 +121,18 @@
     </collision>
   </gazebo>
+  <!-- FRONT CASTER -->
   <link name="front_caster">
     <visual>
-      <geometry><mesh filename="package://gazebo/meshes/f_castor.STL"/></geometry>
-      <material name="silver"><color rgba="0.8 0.8 0.8 1"/></material>
-    </visual>
-    <collision>
-      <geometry><sphere radius="0.05"/></geometry>
+      <geometry>
+        <mesh filename="package://gazebo/meshes/f_castor.STL"/>
+      </geometry>
+      <material name="silver">
+        <color rgba="0.8 0.8 0.8 1"/>
+      </material>
+    </visual>
+    <collision>
+      <geometry>
+        <sphere radius="0.05"/>
+      </geometry>
     </collision>
     <inertial>
@@ -119,11 +146,18 @@
     <origin xyz="0.3075 0.045 -0.0575" rpy="0 0 0"/>
   </joint>
+  <!-- BACK CASTER -->
   <link name="back_caster">
     <visual>
-      <geometry><mesh filename="package://gazebo/meshes/r_castor.STL"/></geometry>
-      <material name="silver"/>
-    </visual>
-    <collision>
-      <geometry><sphere radius="0.05"/></geometry>
+      <geometry>
+        <mesh filename="package://gazebo/meshes/r_castor.STL"/>
+      </geometry>
+      <material name="silver">
+        <color rgba="0.8 0.8 0.8 1"/>
+      </material>
+    </visual>
+    <collision>
+      <geometry>
+        <sphere radius="0.05"/>
+      </geometry>
     </collision>
     <inertial>
@@ -137,5 +171,5 @@
     <origin xyz="-0.3075 -0.045 -0.0575" rpy="0 0 0"/>
   </joint>
-  <!-- Friction for caster links (caster should have contact friction, joints are fixed) -->
+  <!-- CASTER FRICTION -->
   <gazebo reference="front_caster">
     <collision>
@@ -174,4 +208,5 @@
     </collision>
   </gazebo>
+  <!-- IMU -->
   <link name="imu_link"/>
   <joint name="imu_joint" type="fixed">
@@ -188,13 +223,20 @@
     </sensor>
   </gazebo>
+  <!-- LIDAR -->
   <link name="lidar_link">
     <visual>
       <origin xyz="0 0 -0.03" rpy="0 0 0"/>
-      <geometry><mesh filename="package://gazebo/meshes/lidar.STL"/></geometry>
-      <material name="blue"><color rgba="0 0 1 1"/></material>
-    </visual>
-    <collision>
-       <origin xyz="0 0 -0.03" rpy="0 0 0"/>
-      <geometry><cylinder radius="0.055" length="0.0315"/></geometry>
+      <geometry>
+        <mesh filename="package://gazebo/meshes/lidar.STL"/>
+      </geometry>
+      <material name="blue">
+        <color rgba="0 0 1 1"/>
+      </material>
+    </visual>
+    <collision>
+      <origin xyz="0 0 -0.03" rpy="0 0 0"/>
+      <geometry>
+        <cylinder radius="0.055" length="0.0315"/>
+      </geometry>
     </collision>
     <inertial>
@@ -230,8 +272,13 @@
     </sensor>
   </gazebo>
+  <!-- CAMERA BODY -->
   <link name="camera_link">
     <visual>
-      <geometry><box size="0.05 0.05 0.05"/></geometry>
-      <material name="red"><color rgba="1 0 0 1"/></material>
+      <geometry>
+        <mesh filename="package://gazebo/meshes/camera.STL"/>
+      </geometry>
+      <material name="red">
+        <color rgba="1 0 0 1"/>
+      </material>
     </visual>
   </link>
@@ -241,5 +288,6 @@
     <origin xyz="0.25 0 0.1" rpy="0 0 0"/>
   </joint>
-  <link name="camera_link_optical"></link>
+  <!-- CAMERA OPTICAL FRAME -->
+  <link name="camera_link_optical"/>
   <joint name="camera_optical_joint" type="fixed">
     <parent link="camera_link"/>
@@ -267,4 +315,5 @@
     </sensor>
   </gazebo>
+  <!-- GAZEBO PLUGINS: DIFF DRIVE, JOINT STATES, IMU -->
   <gazebo>
     <plugin filename="gz-sim-diff-drive-system" name="gz::sim::systems::DiffDrive">
@@ -278,16 +327,16 @@
       <tf_topic>tf</tf_topic>
       <frame_id>odom</frame_id>
-      <child_frame_id>base_footprint</child_frame_id>
+      <!-- UPDATED: use base_link as child frame -->
+      <child_frame_id>base_link</child_frame_id>
     </plugin>
     <plugin filename="gz-sim-joint-state-publisher-system" name="gz::sim::systems::JointStatePublisher">
       <topic>joint_states</topic>
     </plugin>
-    <!-- <plugin
-      filename="gz-sim-sensors-system"
-      name="gz::sim::systems::Sensors">
+    <!-- Optional Sensors system plugin
+    <plugin filename="gz-sim-sensors-system" name="gz::sim::systems::Sensors">
       <render_engine>ogre2</render_engine>
-    </plugin> -->
-    <plugin filename="gz-sim-imu-system" name="gz::sim::systems::Imu">
     </plugin>
+    -->
+    <plugin filename="gz-sim-imu-system" name="gz::sim::systems::Imu"/>
   </gazebo>
 </robot>

Commit message: Initial commit or updated package

File: urdf/dyno_atman.urdf.xacro (robot description, xacro)
@@ -1,5 +1,5 @@
 <?xml version="1.0"?>
 <robot name="my_mesh_robot" xmlns:xacro="http://www.ros.org/wiki/xacro">
-  <!-- Base footprint -->
+  <!-- base footprint -->
   <link name="base_footprint"/>
   <joint name="base_joint" type="fixed">
@@ -23,7 +23,8 @@
       </geometry>
     </collision>
+    <!-- stable symmetric inertia -->
     <inertial>
       <mass value="40.0"/>
-      <inertia ixx="0.58" ixy="0.0" ixz="0.0" iyy="1.03" iyz="0.0" izz="1.49"/>
+      <inertia ixx="1.0" ixy="0.0" ixz="0.0" iyy="1.0" iyz="0.0" izz="1.0"/>
     </inertial>
   </link>
@@ -46,5 +47,5 @@
     <inertial>
       <mass value="2.4"/>
-      <inertia ixx="0.005" ixy="0" ixz="0" iyy="0.01" iyz="0" izz="0.005"/>
+      <inertia ixx="0.01" ixy="0" ixz="0" iyy="0.01" iyz="0" izz="0.01"/>
     </inertial>
   </link>
@@ -74,5 +75,5 @@
     <inertial>
       <mass value="2.4"/>
-      <inertia ixx="0.005" ixy="0" ixz="0" iyy="0.01" iyz="0" izz="0.005"/>
+      <inertia ixx="0.01" ixy="0" ixz="0" iyy="0.01" iyz="0" izz="0.01"/>
     </inertial>
   </link>
@@ -138,7 +139,8 @@
     <inertial>
       <mass value="0.2"/>
-      <inertia ixx="0.0001" ixy="0" ixz="0" iyy="0.0001" iyz="0" izz="0.0001"/>
-    </inertial>
-  </link>
+      <inertia ixx="0.0005" ixy="0" ixz="0" iyy="0.0005" iyz="0" izz="0.0005"/>
+    </inertial>
+  </link>
+<!-- .................................. -->
   <joint name="front_caster_joint" type="fixed">
     <parent link="base_link"/>
@@ -163,5 +165,5 @@
     <inertial>
       <mass value="0.2"/>
-      <inertia ixx="0.0001" ixy="0" ixz="0" iyy="0.0001" iyz="0" izz="0.0001"/>
+      <inertia ixx="0.0005" ixy="0" ixz="0" iyy="0.0005" iyz="0" izz="0.0005"/>
     </inertial>
   </link>
@@ -208,5 +210,5 @@
     </collision>
   </gazebo>
-  <!-- IMU -->
+  <!-- IMU (with noise / covariance-friendly settings) -->
   <link name="imu_link"/>
   <joint name="imu_joint" type="fixed">
@@ -220,8 +222,24 @@
       <update_rate>100</update_rate>
       <visualize>true</visualize>
+      <!-- topic matches bridge: /imu -->
       <topic>imu</topic>
+      <imu>
+        <!-- simple noise values Nav2/EKF can interpret as non-zero covariance -->
+        <angular_velocity>
+          <noise type="gaussian">
+            <mean>0.0</mean>
+            <stddev>0.001</stddev>
+          </noise>
+        </angular_velocity>
+        <linear_acceleration>
+          <noise type="gaussian">
+            <mean>0.0</mean>
+            <stddev>0.01</stddev>
+          </noise>
+        </linear_acceleration>
+      </imu>
     </sensor>
   </gazebo>
-  <!-- LIDAR -->
+  <!-- LIDAR (topic compatible with /scan bridge) -->
   <link name="lidar_link">
     <visual>
@@ -242,5 +260,5 @@
     <inertial>
       <mass value="0.1"/>
-      <inertia ixx="0.0001" ixy="0" ixz="0" iyy="0.0001" iyz="0" izz="0.0001"/>
+      <inertia ixx="0.0002" ixy="0" ixz="0" iyy="0.0002" iyz="0" izz="0.0002"/>
     </inertial>
   </link>
@@ -253,4 +271,5 @@
     <sensor name="lidar" type="gpu_lidar">
       <pose>0 0 0 0 0 0</pose>
+      <!-- topic matches bridge: /scan -->
       <topic>scan</topic>
       <update_rate>10</update_rate>
@@ -288,16 +307,18 @@
     <origin xyz="0.25 0 0.1" rpy="0 0 0"/>
   </joint>
-  <!-- CAMERA OPTICAL FRAME -->
+  <!-- CAMERA OPTICAL FRAME (standard ROS optical frame: X right, Y down, Z forward) -->
   <link name="camera_link_optical"/>
   <joint name="camera_optical_joint" type="fixed">
     <parent link="camera_link"/>
     <child link="camera_link_optical"/>
-    <origin xyz="0 0 0" rpy="-1.5708 0 -1.5708"/>
-  </joint>
-  <gazebo reference="camera_link">
+    <!-- corrected rotation so image is upright in RViz -->
+    <origin xyz="0 0 0" rpy="0 -1.5708 0"/>
+  </joint>
+  <gazebo reference="camera_link_optical">
     <sensor name="camera" type="camera">
       <pose>0 0 0 0 0 0</pose>
       <visualize>true</visualize>
       <update_rate>30</update_rate>
+      <!-- topic matches bridge: /camera/image_raw -->
       <topic>camera/image_raw</topic>
       <camera>
@@ -327,5 +348,4 @@
       <tf_topic>tf</tf_topic>
       <frame_id>odom</frame_id>
-      <!-- UPDATED: use base_link as child frame -->
       <child_frame_id>base_link</child_frame_id>
     </plugin>
@@ -333,9 +353,4 @@
       <topic>joint_states</topic>
     </plugin>
-    <!-- Optional Sensors system plugin
-    <plugin filename="gz-sim-sensors-system" name="gz::sim::systems::Sensors">
-      <render_engine>ogre2</render_engine>
-    </plugin>
-    -->
     <plugin filename="gz-sim-imu-system" name="gz::sim::systems::Imu"/>
   </gazebo>

Commit message: Updated Gazebo project: added SLAM, worlds, launch scripts, rviz config

File: urdf/dyno_atman.urdf.xacro (robot description, xacro)
@@ -1,12 +1,5 @@
 <?xml version="1.0"?>
 <robot name="my_mesh_robot" xmlns:xacro="http://www.ros.org/wiki/xacro">
-  <!-- base footprint -->
-  <link name="base_footprint"/>
-  <joint name="base_joint" type="fixed">
-    <parent link="base_footprint"/>
-    <child link="base_link"/>
-    <origin xyz="0 0 0.1075" rpy="0 0 0"/>
-  </joint>
-  <!-- BASE LINK -->
+  <!-- base_link IS THE ROOT LINK -->
   <link name="base_link">
     <visual>
@@ -23,5 +16,4 @@
       </geometry>
     </collision>
-    <!-- stable symmetric inertia -->
     <inertial>
       <mass value="40.0"/>
@@ -29,5 +21,5 @@
     </inertial>
   </link>
-  <!-- LEFT WHEEL -->
+  <!-- Left wheel -->
   <link name="left_wheel">
     <visual>
@@ -57,5 +49,5 @@
     <dynamics damping="1.0" friction="0.2"/>
   </joint>
-  <!-- RIGHT WHEEL -->
+  <!-- Right wheel -->
   <link name="right_wheel">
     <visual>
@@ -85,5 +77,4 @@
     <dynamics damping="1.0" friction="0.2"/>
   </joint>
-  <!-- WHEEL FRICTION -->
   <gazebo reference="left_wheel">
     <collision>
@@ -122,5 +113,5 @@
     </collision>
   </gazebo>
-  <!-- FRONT CASTER -->
+  <!-- Front caster -->
   <link name="front_caster">
     <visual>
@@ -142,5 +133,4 @@
     </inertial>
   </link>
-<!-- .................................. -->
   <joint name="front_caster_joint" type="fixed">
     <parent link="base_link"/>
@@ -148,5 +138,5 @@
     <origin xyz="0.3075 0.045 -0.0575" rpy="0 0 0"/>
   </joint>
-  <!-- BACK CASTER -->
+  <!-- Back caster -->
   <link name="back_caster">
     <visual>
@@ -173,5 +163,4 @@
     <origin xyz="-0.3075 -0.045 -0.0575" rpy="0 0 0"/>
   </joint>
-  <!-- CASTER FRICTION -->
   <gazebo reference="front_caster">
     <collision>
@@ -210,5 +199,5 @@
     </collision>
   </gazebo>
-  <!-- IMU (with noise / covariance-friendly settings) -->
+  <!-- IMU -->
   <link name="imu_link"/>
   <joint name="imu_joint" type="fixed">
@@ -222,8 +211,6 @@
       <update_rate>100</update_rate>
       <visualize>true</visualize>
-      <!-- topic matches bridge: /imu -->
       <topic>imu</topic>
       <imu>
-        <!-- simple noise values Nav2/EKF can interpret as non-zero covariance -->
         <angular_velocity>
           <noise type="gaussian">
@@ -241,5 +228,5 @@
     </sensor>
   </gazebo>
-  <!-- LIDAR (topic compatible with /scan bridge) -->
+  <!-- LIDAR -->
   <link name="lidar_link">
     <visual>
@@ -270,6 +257,6 @@
   <gazebo reference="lidar_link">
     <sensor name="lidar" type="gpu_lidar">
+      <gz_frame_id>lidar_link</gz_frame_id>
       <pose>0 0 0 0 0 0</pose>
-      <!-- topic matches bridge: /scan -->
       <topic>scan</topic>
       <update_rate>10</update_rate>
@@ -291,5 +278,5 @@
     </sensor>
   </gazebo>
-  <!-- CAMERA BODY -->
+  <!-- Camera -->
   <link name="camera_link">
     <visual>
@@ -307,10 +294,8 @@
     <origin xyz="0.25 0 0.1" rpy="0 0 0"/>
   </joint>
-  <!-- CAMERA OPTICAL FRAME (standard ROS optical frame: X right, Y down, Z forward) -->
   <link name="camera_link_optical"/>
   <joint name="camera_optical_joint" type="fixed">
     <parent link="camera_link"/>
     <child link="camera_link_optical"/>
-    <!-- corrected rotation so image is upright in RViz -->
     <origin xyz="0 0 0" rpy="0 -1.5708 0"/>
   </joint>
@@ -320,5 +305,4 @@
       <visualize>true</visualize>
       <update_rate>30</update_rate>
-      <!-- topic matches bridge: /camera/image_raw -->
       <topic>camera/image_raw</topic>
       <camera>
@@ -336,5 +320,5 @@
     </sensor>
   </gazebo>
-  <!-- GAZEBO PLUGINS: DIFF DRIVE, JOINT STATES, IMU -->
+  <!-- Gazebo plugins -->
   <gazebo>
     <plugin filename="gz-sim-diff-drive-system" name="gz::sim::systems::DiffDrive">

Commit message: Updated Gazebo project: added SLAM, worlds, launch scripts, maps,  rviz config

File: urdf/dyno_atman.urdf.xacro (robot description, xacro)
@@ -1,5 +1,10 @@
 <?xml version="1.0"?>
 <robot name="my_mesh_robot" xmlns:xacro="http://www.ros.org/wiki/xacro">
-  <!-- base_link IS THE ROOT LINK -->
+  <link name="base_footprint"/>
+  <joint name="base_joint" type="fixed">
+    <parent link="base_footprint"/>
+    <child link="base_link"/>
+    <origin xyz="0 0 0.1075" rpy="0 0 0"/>
+  </joint>
   <link name="base_link">
     <visual>
@@ -21,5 +26,4 @@
     </inertial>
   </link>
-  <!-- Left wheel -->
   <link name="left_wheel">
     <visual>
@@ -49,5 +53,4 @@
     <dynamics damping="1.0" friction="0.2"/>
   </joint>
-  <!-- Right wheel -->
   <link name="right_wheel">
     <visual>
@@ -113,5 +116,4 @@
     </collision>
   </gazebo>
-  <!-- Front caster -->
   <link name="front_caster">
     <visual>
@@ -138,5 +140,4 @@
     <origin xyz="0.3075 0.045 -0.0575" rpy="0 0 0"/>
   </joint>
-  <!-- Back caster -->
   <link name="back_caster">
     <visual>
@@ -199,5 +200,4 @@
     </collision>
   </gazebo>
-  <!-- IMU -->
   <link name="imu_link"/>
   <joint name="imu_joint" type="fixed">
@@ -228,5 +228,4 @@
     </sensor>
   </gazebo>
-  <!-- LIDAR -->
   <link name="lidar_link">
     <visual>
@@ -278,5 +277,4 @@
     </sensor>
   </gazebo>
-  <!-- Camera -->
   <link name="camera_link">
     <visual>
@@ -320,5 +318,4 @@
     </sensor>
   </gazebo>
-  <!-- Gazebo plugins -->
   <gazebo>
     <plugin filename="gz-sim-diff-drive-system" name="gz::sim::systems::DiffDrive">
@@ -332,6 +329,5 @@
       <tf_topic>tf</tf_topic>
       <frame_id>odom</frame_id>
-      <child_frame_id>base_link</child_frame_id>
-    </plugin>
+      <child_frame_id>base_footprint</child_frame_id> </plugin>
     <plugin filename="gz-sim-joint-state-publisher-system" name="gz::sim::systems::JointStatePublisher">
       <topic>joint_states</topic>
